File: Board/Faux Analog Clock.kicad_sch (KiCad schematic)
At the start: 442 parts, among them J1 Barrel_Jack_Switch, J2 AtmegaICSPHeader, J3 Adafruit RTC #3296, J4 Adafruit GPS #746, J5 Aux Board Connector, J6 Select, J7 Enter, SW1 Select, SW2 Enter, U1 ATmega328P-P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

Commit message: Resistor values tweaked
Parts:
- R10, R11, R12, R13, R14, R15, R16, R17, R18, R19, R6, R7, R8, R9: value 100 -> (none)
Changed lines of the file:
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@@
     (in_bom yes) (on_board yes) (fields_autoplaced)
     (property "Reference" "R15" (id 0) (at 189.23 209.55 90))
-    (property "Value" "100" (id 1) (at 189.23 212.09 90))
+    (property "Value" "" (id 1) (at 189.23 212.09 90))
     (property "Footprint" "Resistor_THT:R_Axial_DIN0207_L6.3mm_D2.5mm_P10.16mm_Horizontal" (id 2) (at 189.23 217.678 90)
       (effects (font (size 1.27 1.27)) hide)
@@
     (in_bom yes) (on_board yes) (fields_autoplaced)
     (property "Reference" "R6" (id 0) (at 189.23 95.25 90))
-    (property "Value" "100" (id 1) (at 189.23 97.79 90))
+    (property "Value" "" (id 1) (at 189.23 97.79 90))
     (property "Footprint" "Resistor_THT:R_Axial_DIN0207_L6.3mm_D2.5mm_P10.16mm_Horizontal" (id 2) (at 189.23 103.378 90)
       (effects (font (size 1.27 1.27)) hide)
@@
     (in_bom yes) (on_board yes) (fields_autoplaced)
     (property "Reference" "R11" (id 0) (at 189.23 158.75 90))
-    (property "Value" "100" (id 1) (at 189.23 161.29 90))
+    (property "Value" "" (id 1) (at 189.23 161.29 90))
     (property "Footprint" "Resistor_THT:R_Axial_DIN0207_L6.3mm_D2.5mm_P10.16mm_Horizontal" (id 2) (at 189.23 166.878 90)
       (effects (font (size 1.27 1.27)) hide)
@@
     (in_bom yes) (on_board yes) (fields_autoplaced)
     (property "Reference" "R10" (id 0) (at 189.23 146.05 90))
-    (property "Value" "100" (id 1) (at 189.23 148.59 90))
+    (property "Value" "" (id 1) (at 189.23 148.59 90))
     (property "Footprint" "Resistor_THT:R_Axial_DIN0207_L6.3mm_D2.5mm_P10.16mm_Horizontal" (id 2) (at 189.23 154.178 90)
       (effects (font (size 1.27 1.27)) hide)
@@
     (in_bom yes) (on_board yes) (fields_autoplaced)
     (property "Reference" "R16" (id 0) (at 189.23 222.25 90))
-    (property "Value" "100" (id 1) (at 189.23 224.79 90))
+    (property "Value" "" (id 1) (at 189.23 224.79 90))
     (property "Footprint" "Resistor_THT:R_Axial_DIN0207_L6.3mm_D2.5mm_P10.16mm_Horizontal" (id 2) (at 189.23 230.378 90)
       (effects (font (size 1.27 1.27)) hide)
@@
     (in_bom yes) (on_board yes) (fields_autoplaced)
     (property "Reference" "R9" (id 0) (at 189.23 133.35 90))
-    (property "Value" "100" (id 1) (at 189.23 135.89 90))
+    (property "Value" "" (id 1) (at 189.23 135.89 90))
     (property "Footprint" "Resistor_THT:R_Axial_DIN0207_L6.3mm_D2.5mm_P10.16mm_Horizontal" (id 2) (at 189.23 141.478 90)
       (effects (font (size 1.27 1.27)) hide)
@@
     (in_bom yes) (on_board yes) (fields_autoplaced)
     (property "Reference" "R18" (id 0) (at 189.23 247.65 90))
-    (property "Value" "100" (id 1) (at 189.23 250.19 90))
+    (property "Value" "" (id 1) (at 189.23 250.19 90))
     (property "Footprint" "Resistor_THT:R_Axial_DIN0207_L6.3mm_D2.5mm_P10.16mm_Horizontal" (id 2) (at 189.23 255.778 90)
       (effects (font (size 1.27 1.27)) hide)
@@
     (in_bom yes) (on_board yes) (fields_autoplaced)
     (property "Reference" "R12" (id 0) (at 189.23 171.45 90))
-    (property "Value" "100" (id 1) (at 189.23 173.99 90))
+    (property "Value" "" (id 1) (at 189.23 173.99 90))
     (property "Footprint" "Resistor_THT:R_Axial_DIN0207_L6.3mm_D2.5mm_P10.16mm_Horizontal" (id 2) (at 189.23 179.578 90)
       (effects (font (size 1.27 1.27)) hide)
@@
     (in_bom yes) (on_board yes) (fields_autoplaced)
     (property "Reference" "R7" (id 0) (at 189.23 107.95 90))
-    (property "Value" "100" (id 1) (at 189.23 110.49 90))
+    (property "Value" "" (id 1) (at 189.23 110.49 90))
     (property "Footprint" "Resistor_THT:R_Axial_DIN0207_L6.3mm_D2.5mm_P10.16mm_Horizontal" (id 2) (at 189.23 116.078 90)
       (effects (font (size 1.27 1.27)) hide)
@@
     (in_bom yes) (on_board yes) (fields_autoplaced)
     (property "Reference" "R8" (id 0) (at 189.23 120.65 90))
-    (property "Value" "100" (id 1) (at 189.23 123.19 90))
+    (property "Value" "" (id 1) (at 189.23 123.19 90))
     (property "Footprint" "Resistor_THT:R_Axial_DIN0207_L6.3mm_D2.5mm_P10.16mm_Horizontal" (id 2) (at 189.23 128.778 90)
       (effects (font (size 1.27 1.27)) hide)
@@
     (in_bom yes) (on_board yes) (fields_autoplaced)
     (property "Reference" "R14" (id 0) (at 189.23 196.85 90))
-    (property "Value" "100" (id 1) (at 189.23 199.39 90))
+    (property "Value" "" (id 1) (at 189.23 199.39 90))
     (property "Footprint" "Resistor_THT:R_Axial_DIN0207_L6.3mm_D2.5mm_P10.16mm_Horizontal" (id 2) (at 189.23 204.978 90)
       (effects (font (size 1.27 1.27)) hide)
@@
     (in_bom yes) (on_board yes) (fields_autoplaced)
     (property "Reference" "R19" (id 0) (at 189.23 275.59 90))
-    (property "Value" "100" (id 1) (at 189.23 278.13 90))
+    (property "Value" "" (id 1) (at 189.23 278.13 90))
     (property "Footprint" "Resistor_THT:R_Axial_DIN0207_L6.3mm_D2.5mm_P10.16mm_Horizontal" (id 2) (at 189.23 283.718 90)
       (effects (font (size 1.27 1.27)) hide)
@@
     (in_bom yes) (on_board yes) (fields_autoplaced)
     (property "Reference" "R13" (id 0) (at 189.23 184.15 90))
-    (property "Value" "100" (id 1) (at 189.23 186.69 90))
+    (property "Value" "" (id 1) (at 189.23 186.69 90))
     (property "Footprint" "Resistor_THT:R_Axial_DIN0207_L6.3mm_D2.5mm_P10.16mm_Horizontal" (id 2) (at 189.23 192.278 90)
       (effects (font (size 1.27 1.27)) hide)
@@
     (in_bom yes) (on_board yes) (fields_autoplaced)
     (property "Reference" "R17" (id 0) (at 189.23 234.95 90))
-    (property "Value" "100" (id 1) (at 189.23 237.49 90))
+    (property "Value" "" (id 1) (at 189.23 237.49 90))
     (property "Footprint" "Resistor_THT:R_Axial_DIN0207_L6.3mm_D2.5mm_P10.16mm_Horizontal" (id 2) (at 189.23 243.078 90)
       (effects (font (size 1.27 1.27)) hide)
@@
     )
     (path "/0ddb5b7c-c191-491d-b785-ee9ddc40e98d"
-      (reference "R6") (unit 1) (value "100") (footprint "Resistor_THT:R_Axial_DIN0207_L6.3mm_D2.5mm_P10.16mm_Horizontal")
+      (reference "R6") (unit 1) (value "62") (footprint "Resistor_THT:R_Axial_DIN0207_L6.3mm_D2.5mm_P10.16mm_Horizontal")
     )
     (path "/9dc7217f-30d1-448f-b445-32230cb57a5d"
-      (reference "R7") (unit 1) (value "100") (footprint "Resistor_THT:R_Axial_DIN0207_L6.3mm_D2.5mm_P10.16mm_Horizontal")
+      (reference "R7") (unit 1) (value "62") (footprint "Resistor_THT:R_Axial_DIN0207_L6.3mm_D2.5mm_P10.16mm_Horizontal")
     )
     (path "/a6fc959f-573e-4e96-9a76-059c4a7e1762"
-      (reference "R8") (unit 1) (value "100") (footprint "Resistor_THT:R_Axial_DIN0207_L6.3mm_D2.5mm_P10.16mm_Horizontal")
+      (reference "R8") (unit 1) (value "62") (footprint "Resistor_THT:R_Axial_DIN0207_L6.3mm_D2.5mm_P10.16mm_Horizontal")
     )
     (path "/7fcd3782-f2a8-47a9-9edf-23ee2065abc7"
-      (reference "R9") (unit 1) (value "100") (footprint "Resistor_THT:R_Axial_DIN0207_L6.3mm_D2.5mm_P10.16mm_Horizontal")
+      (reference "R9") (unit 1) (value "62") (footprint "Resistor_THT:R_Axial_DIN0207_L6.3mm_D2.5mm_P10.16mm_Horizontal")
     )
     (path "/52e6f1f2-5bd2-478d-ae36-72ec5ec1856c"
-      (reference "R10") (unit 1) (value "100") (footprint "Resistor_THT:R_Axial_DIN0207_L6.3mm_D2.5mm_P10.16mm_Horizontal")
+      (reference "R10") (unit 1) (value "62") (footprint "Resistor_THT:R_Axial_DIN0207_L6.3mm_D2.5mm_P10.16mm_Horizontal")
     )
     (path "/23330ba2-dd7d-4704-926e-d71d7084cd1d"
-      (reference "R11") (unit 1) (value "100") (footprint "Resistor_THT:R_Axial_DIN0207_L6.3mm_D2.5mm_P10.16mm_Horizontal")
+      (reference "R11") (unit 1) (value "62") (footprint "Resistor_THT:R_Axial_DIN0207_L6.3mm_D2.5mm_P10.16mm_Horizontal")
     )
     (path "/912bf7ea-53b1-4ab9-90b7-5e32db34aff0"
-      (reference "R12") (unit 1) (value "100") (footprint "Resistor_THT:R_Axial_DIN0207_L6.3mm_D2.5mm_P10.16mm_Horizontal")
+      (reference "R12") (unit 1) (value "62") (footprint "Resistor_THT:R_Axial_DIN0207_L6.3mm_D2.5mm_P10.16mm_Horizontal")
     )
     (path "/d18ea326-54ec-42b3-b06e-bd0a82e0ff03"
-      (reference "R13") (unit 1) (value "100") (footprint "Resistor_THT:R_Axial_DIN0207_L6.3mm_D2.5mm_P10.16mm_Horizontal")
+      (reference "R13") (unit 1) (value "62") (footprint "Resistor_THT:R_Axial_DIN0207_L6.3mm_D2.5mm_P10.16mm_Horizontal")
     )
     (path "/bba1584f-73e8-4b82-8f2b-59172f6a5652"
-      (reference "R14") (unit 1) (value "100") (footprint "Resistor_THT:R_Axial_DIN0207_L6.3mm_D2.5mm_P10.16mm_Horizontal")
+      (reference "R14") (unit 1) (value "62") (footprint "Resistor_THT:R_Axial_DIN0207_L6.3mm_D2.5mm_P10.16mm_Horizontal")
     )
     (path "/07a3b87d-5b9a-46f0-8178-60f2fd6810e7"
-      (reference "R15") (unit 1) (value "100") (footprint "Resistor_THT:R_Axial_DIN0207_L6.3mm_D2.5mm_P10.16mm_Horizontal")
+      (reference "R15") (unit 1) (value "62") (footprint "Resistor_THT:R_Axial_DIN0207_L6.3mm_D2.5mm_P10.16mm_Horizontal")
     )
     (path "/619c8661-4b07-4646-82bf-8a9a6e5cd53f"
-      (reference "R16") (unit 1) (value "100") (footprint "Resistor_THT:R_Axial_DIN0207_L6.3mm_D2.5mm_P10.16mm_Horizontal")
+      (reference "R16") (unit 1) (value "62") (footprint "Resistor_THT:R_Axial_DIN0207_L6.3mm_D2.5mm_P10.16mm_Horizontal")
     )
     (path "/dd448503-327a-421c-b9d8-35c81a3b0391"
-      (reference "R17") (unit 1) (value "100") (footprint "Resistor_THT:R_Axial_DIN0207_L6.3mm_D2.5mm_P10.16mm_Horizontal")
+      (reference "R17") (unit 1) (value "62") (footprint "Resistor_THT:R_Axial_DIN0207_L6.3mm_D2.5mm_P10.16mm_Horizontal")
     )
     (path "/8db325b5-4292-4734-87ff-5d68f49dad42"
-      (reference "R18") (unit 1) (value "100") (footprint "Resistor_THT:R_Axial_DIN0207_L6.3mm_D2.5mm_P10.16mm_Horizontal")
+      (reference "R18") (unit 1) (value "62") (footprint "Resistor_THT:R_Axial_DIN0207_L6.3mm_D2.5mm_P10.16mm_Horizontal")
     )
     (path "/bd00bb86-72f0-4d08-b0f5-dfb9eac49b33"
-      (reference "R19") (unit 1) (value "100") (footprint "Resistor_THT:R_Axial_DIN0207_L6.3mm_D2.5mm_P10.16mm_Horizontal")
+      (reference "R19") (unit 1) (value "62") (footprint "Resistor_THT:R_Axial_DIN0207_L6.3mm_D2.5mm_P10.16mm_Horizontal")
     )
     (path "/08ca546a-73ee-4a89-9e96-926e36c5a52c"
